File: MainBoard/CURRENT_MEASURE.sch (KiCad schematic (older format))
At the start: 52 parts

Commit message: R0.1
Parts:
- removed J? (x8): AudioJack2_Ground, symbol Connector:AudioJack2_Ground
- removed R? (x8): 10k, symbol Device:R
- removed U?: 4051, symbol 4xxx:4051
- added C?: 10uF, symbol Device:C
- added C?: 0.1uF, symbol Device:C
- added D?: D_Schottky, symbol Device:D_Schottky
- added Q?: NMOS, symbol Device:Q_NMOS_DGS
- added R?: 400, symbol Device:R
- added R?: 27k, symbol Device:R
- added R?: 220, symbol Device:R
- added U? (x4): MCP6004, symbol Amplifier_Operational:MCP6004
Connections:
- net labels added: +6V, CLR_CURRENT, CUR_PHASE, CUR_VAL
- net labels removed: -3V3, CH_B11, CH_C0, CH_C1, CH_C2, CH_C3, CH_C4, CH_C5, CH_C6, CH_C7, CH_C8, CUR_MUX_OUT, MUX_2, MUX_SEL_4, SZ_B11, SZ_C1, SZ_C2, SZ_C3, SZ_C5, SZ_C6, SZ_C7, SZ_C8
- wire segments 228 -> 200
- no-connect marks 5 -> 9
Other:
- note removed: "NOT FOR MANUFACTURE"
- moved on the sheet: U?

Commit message: Layout Main Board
Layout main PCB
Parts:
- removed J? (x15): AudioJack2_Ground, symbol Connector:AudioJack2_Ground
- removed R? (x16): 10k, symbol Device:R
- removed R?: 400, symbol Device:R
- added C13, C15, C17: 0.1uF, Capacitor_THT:C_Rect_L4.0mm_W2.5mm_P2.50mm, symbol Device:C
- added J16: ADDL_INPUT1, Connector_PinHeader_2.54mm:PinHeader_1x04_P2.54mm_Vertical, symbol Connector:Conn_01x04_Female
- added J17: GND, Connector_PinHeader_2.54mm:PinHeader_1x04_P2.54mm_Vertical, symbol Connector:Conn_01x04_Female
- added J18: ADDL_INPUT2, Connector_PinHeader_2.54mm:PinHeader_1x04_P2.54mm_Vertical, symbol Connector:Conn_01x04_Female
- added J19: PRESCALER, Connector_PinHeader_2.54mm:PinHeader_2x02_P2.54mm_Vertical, symbol Connector_Generic:Conn_02x02_Odd_Even
- added P2: CH1, PanelIQ:DC-005, symbol Connector:Barrel_Jack_Switch
- added P3: CH2, PanelIQ:DC-005, symbol Connector:Barrel_Jack_Switch
- added P4: CH3, PanelIQ:DC-005, symbol Connector:Barrel_Jack_Switch
- added P5: CH4, PanelIQ:DC-005, symbol Connector:Barrel_Jack_Switch
- added P6: CH5, PanelIQ:DC-005, symbol Connector:Barrel_Jack_Switch
- added P7: CH6, PanelIQ:DC-005, symbol Connector:Barrel_Jack_Switch
- added P8: CH7, PanelIQ:DC-005, symbol Connector:Barrel_Jack_Switch
- added R10, R25, R26, R33: 27k, Resistor_THT:R_Axial_DIN0204_L3.6mm_D1.6mm_P7.62mm_Horizontal, symbol Device:R
- added unit 4 of U6
- C14: renamed from C?; footprint (none) -> Capacitor_THT:C_Rect_L4.0mm_W2.5mm_P2.50mm
- C16: renamed from C?; footprint (none) -> Capacitor_THT:CP_Radial_D5.0mm_P2.00mm; P/N (none) -> 732-8625-1-ND
- D5: renamed from D?; value D_Schottky -> SB140TA; footprint (none) -> Diode_THT:D_DO-41_SOD81_P10.16mm_Horizontal; P/N (none) -> SB140TA
- P1: renamed from J?; value AudioJack2_Ground -> CH0; footprint (none) -> PanelIQ:DC-005; symbol Connector:AudioJack2_Ground -> Connector:Barrel_Jack_Switch; P/N (none) -> 103168-1
- Q2: renamed from Q?; value NMOS -> 2N7000; footprint (none) -> Package_TO_SOT_THT:TO-92_Inline; P/N (none) -> 2N7000-D74ZFSCT-ND
- R23: renamed from R?; value 220 -> 330; footprint (none) -> Resistor_THT:R_Axial_DIN0204_L3.6mm_D1.6mm_P7.62mm_Horizontal
- R24: renamed from R?; footprint (none) -> Resistor_THT:R_Axial_DIN0204_L3.6mm_D1.6mm_P7.62mm_Horizontal; P/N (none) -> RNMF14FAD27K0CT-ND
- U5, U7, U8: renamed from U?; footprint (none) -> Package_DIP:DIP-16_W7.62mm_LongPads; P/N (none) -> 296-47632-ND
- U6: renamed from U?; footprint (none) -> Package_DIP:DIP-14_W7.62mm_LongPads
Connections:
- net labels added: ADC_IN, MUX_SELECT0, MUX_SELECT1, MUX_SELECT2, MUX_SELECT3, MUX_SELECT[0..3]
- net labels removed: MUX_SEL_0, MUX_SEL_1, MUX_SEL_2, MUX_SEL_3, SZ_A0, SZ_A1, SZ_A2, SZ_A4, SZ_A5, SZ_A6, SZ_A7, SZ_B0, SZ_B1, SZ_B2, SZ_B3, SZ_B4, SZ_B5, SZ_B6, SZ_B7
- wire segments 200 -> 192
Other:
- note added: "**NOTE SWAPPED 0/2\nMUX SELECT PINS\nFOR LAYOUT PURPOSES"
- moved on the sheet: D5, R24, U5, U6A, U6B, U6C, U7, U8
