File: MainBoard/MOTOR_CONTROL.sch (KiCad schematic (older format))
At the start: 8 parts

Commit message: R0.1
Parts:
- removed C? (x4): C, symbol Device:C
- removed J?: SERVO 1, symbol Connector:Conn_01x03_Male
- removed U?: TMC262, Package_DFN_QFN:QFN-32-1EP_5x5mm_P0.5mm_EP3.45x3.45mm, symbol Driver_Motor:TMC262
- added C? (x5): 0.1uF, symbol Device:C
- added C?: 0.22uF, symbol Device:C
- added C?: 330uF 12V, symbol Device:C
- added J?: SERVO2, symbol Connector:Conn_01x03_Male
- added J?: STEP_DIR, symbol Connector:Conn_01x02_Male
- added R? (x2): 68m, symbol Device:R
- added R?: 100k, symbol Device:R
- added R?: 27k, symbol Device:R
- added R?: 1k, symbol Device:R
- added SW?: SW_DIP_x03, symbol Switch:SW_DIP_x03
- added U?: TMC4210-I, Package_SO:SSOP-16_3.9x4.9mm_P0.635mm, symbol PanelIQ:TMC4210-I
- added U?: A4988, QFN-28_ALM, symbol PanelIQ:A4988
- added X?: ASE-16MHz, Oscillator:Oscillator_SMD_Abracon_ASE-4Pin_3.2x2.5mm, symbol Oscillator:ASE-xxxMHz
- J?: value Conn_01x04_Female -> STEPPER_OUT
Connections:
- net labels added: +3.3V, +6V, HOME_SW
- wire segments 74 -> 136
- no-connect marks 2 -> 1
Other:
- note added: "KEEP TRACES SHORT\nHIGH FREQUENCY"
- note added: "TODO: Figure out \ndoor interlock sleep"
- note removed: "MOTOR DRIVE\nTBD DEPENDING\nON CURRENT\nREQUIREMENTS"
- note removed: "NOT FOR MANUFACTURE"
- moved on the sheet: J?

Commit message: Layout Main Board
Layout main PCB
Parts:
- removed R?: 100k, symbol Device:R
- removed R?: 27k, symbol Device:R
- removed SW?: SW_DIP_x03, symbol Switch:SW_DIP_x03
- added J11: MS SET, Connector_PinHeader_2.54mm:PinHeader_2x03_P2.54mm_Vertical, symbol Connector_Generic:Conn_02x03_Odd_Even
- added J13: DIR, Connector_PinHeader_2.54mm:PinHeader_1x02_P2.54mm_Vertical, symbol Connector:Conn_01x02_Male
- added R28: 27k, Resistor_THT:R_Axial_DIN0204_L3.6mm_D1.6mm_P7.62mm_Horizontal, symbol Device:R
- added R29, R30: 10k, Resistor_THT:R_Axial_DIN0204_L3.6mm_D1.6mm_P7.62mm_Horizontal, symbol Device:R
- C18, C19, C20, C21, C22, C23: renamed from C?; footprint (none) -> Capacitor_THT:C_Rect_L4.0mm_W2.5mm_P2.50mm
- C24: renamed from C?; footprint (none) -> Capacitor_THT:CP_Radial_D8.0mm_P3.50mm; P/N (none) -> 732-8603-1-ND
- J10, J14: renamed from J?; footprint (none) -> Connector_PinHeader_2.54mm:PinHeader_1x03_P2.54mm_Vertical
- J12: renamed from J?; value STEP_DIR -> STEP; footprint (none) -> Connector_PinHeader_2.54mm:PinHeader_1x02_P2.54mm_Vertical
- J15: renamed from J?; footprint (none) -> Connector_JST:JST_XH_B4B-XH-AM_1x04_P2.50mm_Vertical
- R27: renamed from R?; footprint (none) -> Resistor_THT:R_Axial_DIN0204_L3.6mm_D1.6mm_P7.62mm_Horizontal
- R31, R32: renamed from R?; footprint (none) -> Resistor_SMD:R_1206_3216Metric_Pad1.30x1.75mm_HandSolder
- U10: renamed from U?; footprint QFN-28_ALM -> Package_DFN_QFN:QFN-28-1EP_5x5mm_P0.5mm_EP3.35x3.35mm_ThermalVias
- U9: renamed from U?; symbol PanelIQ:TMC4210-I -> MainBoard-rescue:TMC4210-I-PanelIQ
- gave numbers to parts that had none: 1
Connections:
- net labels added: 16MHZ_CLK, DIR_IN, DIR_OUT, MOTOR_A+, MOTOR_A-, MOTOR_B+, MOTOR_B-, MS1, MS2, MS3, SENSE_1, SENSE_2, SPI0, SPI1, SPI2, SPI4, SPI[0..5], STEP_IN, STEP_OUT, VREF, VREG
- net labels removed: CLK, CS_STEP, DIN, DOUT, SPI
- wire segments 136 -> 145
Other:
- note added: "SPI PIN NAMING\n0 - CLK\n1 - MISO\n2 - MOSI\n3 - CS_ADC\n4 - CS_STEP\n5 - CS_SD"
- moved on the sheet: C20, C22, C23, C24, J15, R31, R32

Commit message: Final MainBoard
Parts:
- J15: value STEPPER_OUT -> STEPPER
Changed lines of the file:
@@
 Sheet 5 5
 Title "PanelIQ Main Board - Motor Control"
-Date "2022-02-10"
+Date "2022-02-11"
 Rev "A"
 Comp "Drawn By: Thomas Beckley"
@@
 P 10900 4150
 F 0 "J15" H 10792 3725 50  0000 C CNN
-F 1 "STEPPER_OUT" H 10792 3816 50  0000 C CNN
+F 1 "STEPPER" H 10792 3816 50  0000 C CNN
 F 2 "Connector_JST:JST_XH_B4B-XH-AM_1x04_P2.50mm_Vertical" H 10900 4150 50  0001 C CNN
 F 3 "~" H 10900 4150 50  0001 C CNN
