File: MainBoard/MainBoard.sch (KiCad schematic (older format))
At the start: 32 parts

Commit message: Layout Main Board
Layout main PCB
Parts:
- removed C? (x2): 0.1uF, symbol Device:C
- removed C?: 470uF, symbol Device:CP
- removed C?: 330uF 12V, symbol Device:CP
- removed L?: 10uH, symbol Device:L
- removed R?: 10k, symbol Device:R
- removed SW?: RESET, symbol Switch:SW_Push
- added R4: 27k, Resistor_THT:R_Axial_DIN0204_L3.6mm_D1.6mm_P7.62mm_Horizontal, symbol Device:R
- BZ1: renamed from BZ?; footprint (none) -> Buzzer_Beeper:Buzzer_12x9.5RM7.6; P/N (none) -> 2223-CMI-1295IC-0585T-ND
- C1: renamed from C?; footprint (none) -> Capacitor_THT:CP_Radial_D8.0mm_P3.50mm; P/N (none) -> 732-8603-1-ND
- C2: renamed from C?; value 0.1uF -> 0.22uF; footprint (none) -> Capacitor_THT:C_Rect_L4.0mm_W2.5mm_P2.50mm
- C3: renamed from C?; footprint (none) -> Capacitor_THT:CP_Radial_D13.0mm_P5.00mm; P/N (none) -> 399-ESK478M010AL4AA-ND
- C4: renamed from C?; value 470uF -> 330uF 12V; footprint (none) -> Capacitor_THT:CP_Radial_D8.0mm_P3.50mm; P/N (none) -> 732-8603-1-ND
- C6: renamed from C?; footprint (none) -> Capacitor_THT:C_Rect_L4.0mm_W2.5mm_P2.50mm
- D1: renamed from D?; value D_Schottky -> SB140TA; footprint (none) -> Diode_THT:D_DO-41_SOD81_P10.16mm_Horizontal; P/N (none) -> SB140TA
- J1, J2: renamed from J?; footprint (none) -> Connector_Pin:Pin_D1.4mm_L8.5mm_W2.8mm_FlatFork
- J3: renamed from J?; value DOOR -> DOOR_JMPR; footprint (none) -> Connector_PinHeader_2.54mm:PinHeader_1x02_P2.54mm_Vertical
- J4, J5: renamed from J?; footprint (none) -> Connector_PinHeader_2.54mm:PinHeader_1x02_P2.54mm_Vertical
- J6: renamed from J?; footprint (none) -> Connector_Card:microSD_HC_Wuerth_693072010801
- L1: renamed from L?; value 109uH -> 150uH; footprint (none) -> Inductor_THT:L_Radial_D6.0mm_P4.00mm
- Q1: renamed from Q?; value Q_NMOS_DGS -> 2N7000; footprint (none) -> Package_TO_SOT_THT:TO-92_Inline; P/N (none) -> 2N7000-D74ZFSCT-ND
- R1, R6: renamed from R?; value R -> 10k; footprint (none) -> Resistor_THT:R_Axial_DIN0204_L3.6mm_D1.6mm_P7.62mm_Horizontal
- R2, R8, R9: renamed from R?; footprint (none) -> Resistor_THT:R_Axial_DIN0204_L3.6mm_D1.6mm_P7.62mm_Horizontal
- R3: renamed from R?; value 68k -> 27k; footprint (none) -> Resistor_THT:R_Axial_DIN0204_L3.6mm_D1.6mm_P7.62mm_Horizontal; P/N (none) -> RNMF14FAD27K0CT-ND
- R5: renamed from R?; value 6k2 -> 10k; footprint (none) -> Resistor_THT:R_Axial_DIN0204_L3.6mm_D1.6mm_P7.62mm_Horizontal
- R7: renamed from R?; value 33k -> 27k; footprint (none) -> Resistor_THT:R_Axial_DIN0204_L3.6mm_D1.6mm_P7.62mm_Horizontal; P/N (none) -> RNMF14FAD27K0CT-ND
- U1: renamed from U?; symbol PanelIQ:MC33167THG -> MainBoard-rescue:MC33167THG-PanelIQ
- U2: renamed from U?; footprint MODULE_ESP32-DEVKITC-32U -> PanelIQ:MODULE_ESP32-DEVKITC-32U; symbol PanelIQ:ESP32-DEVKITC-32U -> MainBoard-rescue:ESP32-DEVKITC-32U-PanelIQ
Connections:
- net labels added: CLR_CURRENT, DOOR_OUT, HOME_OUT, LED_OUT, MUX_SELECT0, MUX_SELECT1, MUX_SELECT2, MUX_SELECT3, MUX_SELECT[0..3], SPI0, SPI1, SPI2, SPI3, SPI4, SPI5, SPI[0..5]
- net labels removed: CLK, CS_ADC, CS_SD, CS_STEP, DIN, DOUT, EN, MUX_SEL, MUX_SEL_0, MUX_SEL_1, MUX_SEL_2, MUX_SEL_3, SPI
- wire segments 131 -> 109
- no-connect marks 10 -> 15
Other:
- note added: "SPI PIN NAMING\n0 - CLK\n1 - MISO\n2 - MOSI\n3 - CS_ADC\n4 - CS_STEP\n5 - CS_SD"
- note added: "VREF = 5.05V\nVo*54/(10+54) = 5.05\nVo = 5.985V"
- note removed: "TODO: CLC FILTER MATH"
- note removed: "VREF = 5.05V\nVo*33/(33+6.2) = 5.05\nVo = 5.998V"
- moved on the sheet: C1, C2, C3, C4, D1, J1, J2, J3, J4, J5, L1, R1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

Commit message: Final MainBoard
Parts:
- J3: value DOOR_JMPR -> DOOR
- U2: symbol MainBoard-rescue:ESP32-DEVKITC-32U-PanelIQ -> MainBoard-rescue:ESP32-DEVKITC-32U-PanelIQ-MainBoard-rescue
Connections:
- net CLR_CURRENT: now also U2.11 (IO27); no longer U2.10 (IO26)
- net CUR_PHASE: now also U2.6 (IO35); no longer U2.9 (IO25)
- net MUX_SELECT0: now also U2.9 (IO25); no longer U2.7 (IO32)
- net MUX_SELECT1: now also U2.10 (IO26); no longer U2.8 (IO33)
- net MUX_SELECT2: now also U2.7 (IO32); no longer U2.5 (IO34)
- net MUX_SELECT3: now also U2.8 (IO33); no longer U2.6 (IO35)
- no-connect marks 15 -> 16
Changed lines of the file:
@@
 Sheet 1 5
 Title "PanelIQ Main Board"
-Date "2022-02-10"
+Date "2022-02-11"
 Rev "A"
 Comp "Drawn By: Thomas Beckley"
@@
 Text Label 5350 1850 2    50   ~ 0
 SPI[0..5]
-Text Label 6500 2350 0    50   ~ 0
+Text Label 6500 2550 0    50   ~ 0
 MUX_SELECT[0..3]
 Wire Wire Line
@@
 $EndComp
 $Comp
-L MainBoard-rescue:ESP32-DEVKITC-32U-PanelIQ U2
-U 1 1 626E8F65
-P 8850 2650
-F 0 "U2" H 8850 3817 50  0000 C CNN
-F 1 "ESP32-DEVKITC-32U" H 8850 3726 50  0000 C CNN
-F 2 "PanelIQ:MODULE_ESP32-DEVKITC-32U" H 8400 3700 50  0001 L BNN
-F 3 "https://www.espressif.com/sites/default/files/documentation/esp32_datasheet_en.pdf" H 8850 2650 50  0001 L BNN
-	1    8850 2650
-	1    0    0    -1
-$EndComp
-$Comp
 L power:+6V #PWR018
 U 1 1 626F135E
@@
 NoConn ~ 8300 5600
 Wire Wire Line
-	7300 2450 8150 2450
+	7300 2650 8150 2650
 Text Label 10350 2850 2    50   ~ 0
 SPI0
 Wire Wire Line
-	7300 2150 8150 2150
-Entry Wire Line
-	7300 2150 7200 2050
+	7300 2350 8150 2350
+Entry Wire Line
+	7300 2350 7200 2250
+Text Label 7600 2550 0    50   ~ 0
+MUX_SELECT0
+Text Label 7600 2650 0    50   ~ 0
+MUX_SELECT1
+Text Label 7600 2450 0    50   ~ 0
+MUX_SELECT3
 Text Label 7600 2350 0    50   ~ 0
-MUX_SELECT0
-Text Label 7600 2450 0    50   ~ 0
-MUX_SELECT1
-Text Label 7600 2250 0    50   ~ 0
-MUX_SELECT3
-Text Label 7600 2150 0    50   ~ 0
 MUX_SELECT2
 Wire Wire Line
-	8150 2350 7300 2350
-Wire Wire Line
-	8150 2250 7300 2250
+	8150 2550 7300 2550
+Wire Wire Line
+	8150 2450 7300 2450
+Entry Wire Line
+	7300 2650 7200 2550
 Entry Wire Line
 	7300 2450 7200 2350
 Entry Wire Line
-	7300 2250 7200 2150
-Entry Wire Line
-	7300 2350 7200 2250
+	7300 2550 7200 2450
 Entry Wire Line
 	7650 5300 7550 5200
@@
 P 2700 3650
 F 0 "J3" H 2600 3650 50  0000 C CNN
-F 1 "DOOR_JMPR" H 2750 3500 50  0000 C CNN
+F 1 "DOOR" H 2750 3500 50  0000 C CNN
 F 2 "Connector_PinHeader_2.54mm:PinHeader_1x02_P2.54mm_Vertical" H 2700 3650 50  0001 C CNN
 F 3 "~" H 2700 3650 50  0001 C CNN
@@
 	4950 2150 5650 2150
 Wire Bus Line
-	6500 2350 7200 2350
+	6500 2550 7200 2550
 Text Label 5850 1450 2    50   ~ 0
 MUX_SELECT[0..3]
@@
 	9550 1950 10350 1950
 Wire Wire Line
-	7500 2650 8150 2650
-Text Label 7500 2650 0    50   ~ 0
+	7500 2750 8150 2750
+Text Label 7500 2750 0    50   ~ 0
 CLR_CURRENT
-Text Label 7500 2550 0    50   ~ 0
+Text Label 7600 2250 0    50   ~ 0
 CUR_PHASE
 Text Label 7650 3150 0    50   ~ 0
 LINE_PHASE
 Wire Wire Line
-	8150 2550 7500 2550
+	8150 2250 7600 2250
 Text Label 7850 2950 0    50   ~ 0
 BUZZ
@@
 Wire Wire Line
 	7850 2950 8150 2950
-NoConn ~ 8150 2750
 NoConn ~ 9550 2750
+NoConn ~ 8150 2150
+$Comp
+L MainBoard-rescue:ESP32-DEVKITC-32U-PanelIQ-MainBoard-rescue U2
+U 1 1 626E8F65
+P 8850 2650
+F 0 "U2" H 8850 3817 50  0000 C CNN
+F 1 "ESP32-DEVKITC-32U" H 8850 3726 50  0000 C CNN
+F 2 "PanelIQ:MODULE_ESP32-DEVKITC-32U" H 8400 3700 50  0001 L BNN
+F 3 "https://www.espressif.com/sites/default/files/documentation/esp32_datasheet_en.pdf" H 8850 2650 50  0001 L BNN
+	1    8850 2650
+	1    0    0    -1
+$EndComp
+NoConn ~ 9550 3250
 Wire Bus Line
-	7200 2050 7200 2350
+	7200 2250 7200 2550
 Wire Bus Line
 	7550 4750 7550 5400
